Commit message: Imported upstream version '1.0.14' of 'upstream'

File: roch_description/urdf/roch.urdf.xacro (robot description, xacro)
@@ -133,5 +133,5 @@
     </link>
     <joint name="imu_joint" type="fixed">
-      <origin xyz=" 0.145 0 0.0095" rpy=" 0 -1.5708 3.1416" />
+      <origin xyz=" 0.145 0 0.0095" rpy=" 0 0 3.1415926" />
       <parent link="base_link" />
       <child link="imu_link" />

File: roch_description/urdf/sensors/rplidar.urdf.xacro (robot description, xacro)
@@ -63,5 +63,5 @@
     <link name="base_laser"/>
     <joint name="base_laser_joint" type="fixed">
-      <origin xyz="0 0 0.04076" rpy=" 0 0 ${M_PI/4*3}" />
+      <origin xyz="0 0 0.04076" rpy=" 0 0 2.2689" />
       <parent link="base_laser_link" />
       <child link="base_laser" />
