Commit message: Imported upstream version '1.0.15' of 'upstream'

File: roch_description/urdf/roch_properties.urdf.xacro (robot description, xacro)
@@ -40,8 +40,8 @@
   <property name="r200_op" value="0" />
   <property name="r200_oy" value="0" />
-<!-- Intel R200 param -->
-  <property name="astra_px" value="-0.15" />
-  <property name="astra_py" value="-0.065" />
-  <property name="astra_pz" value="0.725" />
+<!-- Orbbec Astra param -->
+  <property name="astra_px" value="-0.12" />
+  <property name="astra_py" value="0.0" />
+  <property name="astra_pz" value="0.715" />
   <property name="astra_or" value="0" />
   <property name="astra_op" value="0" />

File: roch_description/urdf/sensors/astra.urdf.xacro (robot description, xacro)
@@ -3,35 +3,24 @@
   <xacro:include filename="$(find roch_description)/urdf/roch_gazebo.urdf.xacro"/>
   <xacro:include filename="$(find roch_description)/urdf/roch_properties.urdf.xacro"/>
-  <xacro:property name="astra_cam_py" value="-0.0125"/>
+  <xacro:property name="astra_cam_py" value="0.0125"/>
   <!-- Parameterised in part by the values in roch_properties.urdf.xacro -->
   <xacro:macro name="sensor_astra" params="parent">
     <joint name="camera_rgb_joint" type="fixed">
-      <origin xyz="${astra_px} ${astra_cam_py} ${astra_pz}" rpy="${astra_or} ${astra_op} ${astra_oy}"/>
+      <origin xyz="${astra_px} ${astra_py} ${astra_pz}" rpy="${astra_or} ${astra_op} ${astra_oy}"/>
       <parent link="${parent}"/>
-      <child link="camera_rgb_frame" />
+      <child link="camera_link" />
     </joint>
-    <link name="camera_rgb_frame"/>
-    <joint name="camera_rgb_optical_joint" type="fixed">
-      <origin xyz="0 0 0" rpy="${-M_PI/2} 0 ${-M_PI/2}" />
-      <parent link="camera_rgb_frame" />
-      <child link="camera_rgb_optical_frame" />
-    </joint>
-    <link name="camera_rgb_optical_frame"/>
-    <joint name="camera_joint" type="fixed">
-      <origin xyz="0 ${-astra_cam_py} 0.01" rpy="0 0 0"/>
-      <parent link="camera_rgb_frame"/>
-      <child link="camera_link"/>
-    </joint>
-      <link name="camera_link">
+    <link name="camera_link">
       <visual>
-       <origin xyz="0 0 0" rpy="${M_PI/2} 0 ${M_PI/2}"/>
+       <origin xyz="0 0 0" rpy="1.5707963 0 1.5707963"/>
         <geometry>
-         <mesh filename="package://roch_description/meshes/sensors/astra.dae"/>
+         <mesh filename="package://roch_description/meshes/sensors/astra.dae" scale="0.5 0.5 0.5" />
         </geometry>
+	    <xacro:insert_block name="roch_black"/>
       </visual>
   	  <collision>
-        <origin xyz="0.0 0.0 0.0" rpy="0 0 0"/>
-  	    <geometry>
-  	      <box size="0.07271 0.27794 0.073"/>
+        <origin xyz="0.0 0.0 0.0" rpy="1.5707963 0 1.5707963"/>
+  	    <geometry>.
+         <mesh filename="package://roch_description/meshes/sensors/astra.dae" scale="0.5 0.5 0.5" />
   	    </geometry>
   	  </collision>
@@ -44,9 +33,21 @@
       </inertial>
     </link>
+    <joint name="camera_joint" type="fixed">
+      <origin xyz="0.025 ${astra_cam_py} 0.01  " rpy="0 0 0"/>
+      <parent link="camera_link"/>
+      <child link="camera_rgb_frame"/>
+    </joint>
+    <link name="camera_rgb_frame"/>
+    <joint name="camera_rgb_optical_joint" type="fixed">
+      <origin xyz="0 0 0" rpy="${-M_PI/2} 0 ${-M_PI/2}" />
+      <parent link="camera_rgb_frame" />
+      <child link="camera_rgb_optical_frame" />
+    </joint>
+    <link name="camera_rgb_optical_frame"/>
     <!-- The fixed joints & links below are usually published by static_transformers launched by the OpenNi launch
          files. However, for Gazebo simulation we need them, so we add them here.
          (Hence, don't publish them additionally!) -->
 	<joint name="camera_depth_joint" type="fixed">
-	  <origin xyz="0 ${2 * -astra_cam_py} 0" rpy="0 0 0" />
+	  <origin xyz="0 ${-0.03 -astra_cam_py} 0" rpy="0 0 0" />
 	  <parent link="camera_rgb_frame" />
 	  <child link="camera_depth_frame" />
@@ -59,5 +60,5 @@
 	</joint>
 	<link name="camera_depth_optical_frame"/>
-	<!-- Kinect sensor for simulation -->
+	<!-- astra sensor for simulation -->
 	<roch_sim_3dsensor/>
   </xacro:macro>
